File: wotcher-pcb/wotcher.kicad_pcb (KiCad board)
At the start: 4 copper layers, 41.6 x 39.7 mm, 105 parts, among them CN1 SM02B-SRSS-TB, SW1 SKTDLHE010, SW2 SKTDLHE010, SW3 SKTDLHE010, SW4 SKTDLHE010, U1 KCSA02-105, U2 KCSA02-105, U3 LIS2DW12TR-MS, U5 ATtiny1616-M, U6 KCSA02-105, U7 IS31FL3731-QF, U8 KCSA02-105, U9 DS3231MZ+

Commit message: re-wired something
Connections:
- R2 pad 2: Net-(U3-SDO) -> Net-(U3-SCx)
- R3 pad 2: Net-(U5-PB1) -> Net-(U3-SDx)
- U3 pad 1: Net-(U3-SDO) -> ATtinyVCC
- U3 pad 12: PA6 -> Net-(U3-SCx)
- U3 pad 2: ATtinyVCC -> Net-(U3-SDx)
- U3 pad 4: Net-(U5-PB1) -> unconnected-(U3-NC-Pad4)
- U3 pad 5: ATtinyGND -> PA6
- U3 pad 6: ATtinyGND -> unconnected-(U3-INT2-Pad6)
- U3 pad 7: ATtinyGND -> ATtinyVCC
- U3 pad 9: ATtinyVCC -> ATtinyGND
- U5 pad 13: Net-(U5-PB1) -> Net-(U3-SDx)
- U5 pad 14: Net-(U3-SDO) -> Net-(U3-SCx)
- U7 pad 19: Net-(U5-PB1) -> Net-(U3-SDx)
- U7 pad 20: Net-(U3-SDO) -> Net-(U3-SCx)
- U9 pad 7: Net-(U5-PB1) -> Net-(U3-SDx)
- U9 pad 8: Net-(U3-SDO) -> Net-(U3-SCx)
Routing:
- net Net-(U3-SDx): track 0.00 -> 74.5 mm, vias 0 -> 6
- net Net-(U5-PB1): track 62.9 -> 0.00 mm, vias 7 -> 0
- net Net-(U3-SDO): track 58.4 -> 0.00 mm, vias 3 -> 0
- net Net-(U3-SCx): track 0.00 -> 47.4 mm, vias 0 -> 5
- net ATtinyVCC: track 133.4 -> 139.5 mm, vias 10 -> 12
- net CA3: track 127.5 -> 132.3 mm
- net CA5: track 127.5 -> 130.3 mm
- net Net-(U5-PC3): track 36.1 -> 37.5 mm
- net ATtinyGND: track 90.0 -> 91.2 mm, vias 22 -> 21
- net CA1: track 94.6 -> 95.6 mm
- net PA0: track 31.7 -> 32.6 mm
- net Net-(W61-K): track 39.3 -> 38.4 mm
- net PA6: track 8.48 -> 8.46 mm, vias 3 -> 2

Commit message: no more bitmap D:
Parts:
- added G***: LOGO, LOGO, F.Cu at (65.8, 35.8)
Routing:
- net ATtinyVCC: track 139.5 -> 141.8 mm
- net CA5: track 130.3 -> 129.1 mm
- net Net-(U3-SDx): track 74.5 -> 73.7 mm
- net Net-(U7-R_EXT): track 8.78 -> 8.20 mm
- net CA8: track 121.2 -> 121.7 mm

Commit message: remove backups, and update board again
Parts:
- removed G***: LOGO, LOGO
